File: KiCAD/ETX60.kicad_sch (KiCad schematic)
At the start: 71 parts, among them Q1 Q_NPN_BCE, Q1A IRF9956PbF, Q2 Q_NPN_BCE, Q2A IRF9953PbF, Q3 UnknownIR-Reciever-for-D1-AZ, Q3A IRF9956PbF, Q4 Q_NPN_BCE, Q4A IRF9953PbF, Q5 Q_NPN_BCE, Q6 UnknownIR-Reciever-for-D2-ALT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

Commit message: Version 1.2
Parts:
- C4, C5: value (none) -> 100nF
- D1, D2: value IR -> (none)
- R15, R16, R19, R2, R4, R5: value (none) -> 10k
- U1: value (none) -> PIC16C57C-SO
- X1: value (none) -> 20MHz
Connections:
- net GND^{a} renamed GND^{1}
- net GND^{b} renamed GND^{2}
- net MOT-1a renamed MOT-1A
- net MOT-1b renamed MOT-1B
- net MOT-2a renamed MOT-2A
- net MOT-2b renamed MOT-2B
- net Q2A-G1_Q1C renamed Q2A-G1_Q1c
- net Q2A-G2_Q2C renamed Q2A-G2_Q2c
- net Q4A-G1_Q4C renamed Q4A-G1_Q4c
- net Q4A-G2_Q5C renamed Q4A-G2_Q5c
- net VBAT^{a} renamed VBAT^{1}
- net VBAT^{b} renamed VBAT^{2}
- net VCC^{a} renamed VCC^{1}
- net VCC^{b} renamed VCC^{2}
- net VCC^{c} renamed VCC^{3}
